Commit message: Added functionality to THOR
Redid URDF, allowed control of THOR over ROS, added navigation and utility packages, added launch script

File: thor_description/urdf/thor.urdf.xacro (robot description, xacro)
@@ -16,5 +16,5 @@
   -->
   <!-- Fixed odom dummy frame -->
-  <link name="odom" />
+  <link name="$(arg robot_name)_odom" />
   <!--
     IMPORTS
@@ -30,6 +30,6 @@
   -->
   <!-- Define macros for swerve import -->
-  <xacro:thor name="$(arg robot_name)" parent="odom" hardware_interface="$(arg hardware_interface)">
-	  <origin xyz="0 0 0.053975" rpy="0 0 0"/> <!-- rotate 90 degrees due to error in black box model -->
+  <xacro:thor name="$(arg robot_name)" parent="$(arg robot_name)_odom" hardware_interface="$(arg hardware_interface)">
+	  <origin xyz="0 0 0.053975" rpy="0 0 0"/>
   </xacro:thor>
   <xacro:thor_sensors name="thor"/>

File: thor_description/urdf/thor.xacro (robot description, xacro)
@@ -30,14 +30,6 @@
       LEFT WHEEL DEFINITION
     -->
-    <xacro:motor_joint joint_name="${name}_left_motor_joint" parent="${name}_body" child="${name}_left_motor"
-      x="0.0697624" y="0.1208321" theta="2.61799" hardware_interface="${hardware_interface}"/>
-    <link name="${name}_left_motor">
-      <inertial>
-        <xacro:insert_block name="motor_inertial_properties" />
-      </inertial>
-      <xacro:insert_block name="motor_visual_collision" />
-    </link>
-    <xacro:wheel_joint joint_name="${name}_left_wheel_joint" parent="${name}_left_motor" child="${name}_left_wheel"
-      hardware_interface="${hardware_interface}"/>
+    <xacro:wheel_joint joint_name="${name}_left_wheel_joint" parent="${name}_body" child="${name}_left_wheel"
+      x="0.09226" y="0.1598" theta="2.61799" hardware_interface="${hardware_interface}"/>
     <link name="${name}_left_wheel">
       <inertial>
@@ -49,14 +41,6 @@
       RIGHT WHEEL DEFINITION
     -->
-    <xacro:motor_joint joint_name="${name}_right_motor_joint" parent="${name}_body" child="${name}_right_motor"
-      x="0.0697624" y="-0.1208321" theta="0.523599" hardware_interface="${hardware_interface}"/>
-    <link name="${name}_right_motor">
-      <inertial>
-        <xacro:insert_block name="motor_inertial_properties" />
-      </inertial>
-      <xacro:insert_block name="motor_visual_collision" />
-    </link>
-    <xacro:wheel_joint joint_name="${name}_right_wheel_joint" parent="${name}_right_motor" child="${name}_right_wheel"
-      hardware_interface="${hardware_interface}"/>
+    <xacro:wheel_joint joint_name="${name}_right_wheel_joint" parent="${name}_body" child="${name}_right_wheel"
+      x="0.09226" y="-0.1598" theta="0.523599" hardware_interface="${hardware_interface}"/>
     <link name="${name}_right_wheel">
       <inertial>
@@ -68,14 +52,6 @@
       TAIL WHEEL DEFINITION
     -->
-    <xacro:motor_joint joint_name="${name}_tail_motor_joint" parent="${name}_body" child="${name}_tail_motor"
-      x="-0.1395249" y="0" theta="4.71239" hardware_interface="${hardware_interface}"/>
-    <link name="${name}_tail_motor">
-      <inertial>
-        <xacro:insert_block name="motor_inertial_properties" />
-      </inertial>
-      <xacro:insert_block name="motor_visual_collision" />
-    </link>
-    <xacro:wheel_joint joint_name="${name}_tail_wheel_joint" parent="${name}_tail_motor" child="${name}_tail_wheel"
-      hardware_interface="${hardware_interface}"/>
+    <xacro:wheel_joint joint_name="${name}_tail_wheel_joint" parent="${name}_body" child="${name}_tail_wheel"
+      x="-0.18452" y="0" theta="4.71239" hardware_interface="${hardware_interface}"/>
     <link name="${name}_tail_wheel">
       <inertial>
@@ -101,4 +77,18 @@
       <xacro:insert_block name="lidar_visual_collision" />
     </link>
+    <joint name="${name}_imu_joint" type="fixed">
+      <origin xyz="-0.07378 0.03088 0.04318" rpy="${pi} 0 -${pi/2}" />
+      <parent link="${name}_body" />
+      <child link="${name}_imu" />
+      <axis xyz="0 0 " />
+    </joint>
+    <link name="${name}_imu">
+      <inertial>
+        <mass value="0.001" />
+        <origin xyz="0 0 0" />
+        <inertia ixx="0.0001" ixy="0.0" ixz="0.0" iyy="0.0001" iyz="0.0" izz="0.0001" />
+      </inertial>
+      <!-- <xacro:insert_block name="imu_visual_collision" /> -->
+    </link>
     <!-- <xacro:sick_tim551 name="${name}_laser" ros_topic="scan" height="0.0511"/> -->
   </xacro:macro>

File: thor_description/urdf/thor_utilities.xacro (robot description, xacro)
@@ -8,5 +8,4 @@
 <robot name="thor" xmlns:xacro="http://ros.org/wiki/xacro">
   <!-- Constants -->
-  <xacro:property name="pi" value="3.14159" />
   <xacro:property name="chassis_mass" value="1.666" />
   <xacro:property name="motor_mass" value="0.22578" />
@@ -16,15 +15,10 @@
   <xacro:property name="chassis_geometry">
     <geometry>
-      <mesh filename="package://thor_description/meshes/chassis.stl" />
-    </geometry>
-  </xacro:property>
-  <xacro:property name="motor_geometry">
-    <geometry>
-      <mesh filename="package://thor_description/meshes/motor.stl" />
+      <mesh filename="package://thor_description/meshes/chassis_coarse.stl" />
     </geometry>
   </xacro:property>
   <xacro:property name="wheel_geometry">
     <geometry>
-      <mesh filename="package://thor_description/meshes/wheel.stl" />
+      <mesh filename="package://thor_description/meshes/wheel_coarse.stl" />
     </geometry>
   </xacro:property>
@@ -37,9 +31,4 @@
     <geometry>
       <cylinder length="0.0762" radius="0.2"/>
-    </geometry>
-  </xacro:property>
-  <xacro:property name="motor_collision_geometry">
-    <geometry>
-      <box size="0.0376 0.08682 0.03865"/>
     </geometry>
   </xacro:property>
@@ -82,15 +71,4 @@
     </collision>
   </xacro:property>
-  <xacro:property name="motor_visual_collision">
-    <visual>
-      <origin xyz="0 0 0" rpy="0 0 0" />
-      <xacro:insert_block name="motor_geometry" />
-      <xacro:insert_block name="color_green" />
-    </visual>
-    <collision>
-      <origin xyz="0 0.0265 -0.0095" rpy="0 0 0" />
-      <xacro:insert_block name="motor_collision_geometry" />
-    </collision>
-  </xacro:property>
   <xacro:property name="wheel_visual_collision">
     <visual>
@@ -116,37 +94,15 @@
   </xacro:property>
   <!-- Common link/joint properties -->
-  <xacro:property name="motor_inertial_properties">
-    <origin xyz="0 0 0" rpy="0 0 0" />
-    <mass value="${motor_mass}" />
-    <inertia ixx="0.0002675" ixy="0.0000101" ixz="-0.0000022" iyy="0.0000424" iyz="-0.0000368" izz="0.0002573" />
-  </xacro:property>
   <xacro:property name="wheel_inertial_properties">
         <origin xyz="0 0 0" rpy="0 0 0" />
         <mass value="${wheel_mass}" />
-        <inertia ixx="0.0002079" ixy="0.0000046" ixz="0.0000001" iyy="0.0003299" iyz="-0.0000059" izz="0.0002115" />
+        <inertia ixx="0.00026" ixy="0" ixz="0" iyy="0.00038" iyz="0" izz="0.00026" />
   </xacro:property>
-  <xacro:macro name="motor_joint" params="joint_name parent child x y theta hardware_interface">
+  <xacro:macro name="wheel_joint" params="joint_name parent child x y theta hardware_interface">
     <joint name="${joint_name}" type="continuous">
       <origin xyz="${x} ${y} -0.00445" rpy="0 0 ${theta}" />
       <parent link="${parent}" />
       <child link="${child}" />
-    </joint>
-    <transmission name="${joint_name}_trans">
-      <type>transmission_interface/SimpleTransmission</type>
-      <joint name="${joint_name}">
-        <hardwareInterface>hardware_interface/${hardware_interface}</hardwareInterface>
-      </joint>
-      <actuator name="${joint_name}_motor">
-        <mechanicalReduction>${mechanical_reduction}</mechanicalReduction>
-        <hardwareInterface>hardware_interface/${hardware_interface}</hardwareInterface>
-      </actuator>
-    </transmission>
-  </xacro:macro>
-  <xacro:macro name="wheel_joint" params="joint_name parent child hardware_interface">
-    <joint name="${joint_name}" type="continuous">
-      <origin xyz="0 -0.045 0" rpy="0 0 0" />
-      <parent link="${parent}" />
-      <child link="${child}" />
-      <axis xyz="0 1 0" />
+      <axis xyz="0 -1 0" />
     </joint>
     <transmission name="${joint_name}_trans">
